File: pcb/esp32board/esp32board.kicad_pcb (KiCad board)
At the start: 2 copper layers, 122.2 x 54.6 mm, 89 parts, among them J1 1Wire, J10 NTC5, J11 FuelLevel, J12 12V In, J13 Oil Pressure, J14 Engine, J15 Flywheel, J16 Relays, J5 CAN, J6 NTC1, J7 NTC2, J8 NTC3, J9 NTC4, Q1 BS170F, Q2 BS170F, U1 ESP32-C3-Waveshare, U2 AMS1117-5.0, U3 TJA1050, U4 ADS1115IDGS, U5 ADS1115IDGS, U6 ADS1115IDGS, U7 LM393

Commit message: Fixed some hardware problems, new board
Parts:
- removed D10, D11: LED, LED_SMD:LED_0805_2012Metric_Pad1.15x1.40mm_HandSolder
- removed REF** (x4): MountingHole_3.2mm_M3, MountingHole:MountingHole_3.2mm_M3
- added J2: V2_spare, Connector_PinHeader_2.54mm:PinHeader_1x01_P2.54mm_Vertical, F.Cu at (139.1, 121.4)
- D1: value LED -> SMAJ16CA; footprint LED_SMD:LED_0805_2012Metric_Pad1.15x1.40mm_HandSolder -> Diode_SMD:D_SMA
- Q1, Q2: value BS170F -> BSS138
- R35: value 2K2 -> 1K
- R36: value 3K3 -> 22K
- R42: value 4K7 -> 3K3
- moved D1 99.2 mm to (91.3, 150.0)
- moved C4 72.2 mm to (104.5, 126.5), turned to 90 degrees
- moved C1 48.6 mm to (154.7, 121.8), turned to 180 degrees
- moved U1 41.6 mm to (174.0, 129.5), turned to -90 degrees
- moved U3 39.3 mm to (164.1, 121.4)
- moved R5 37.8 mm to (146.7, 126.5), turned to -90 degrees
- moved R11 36.1 mm to (142.4, 126.5), turned to -90 degrees
- moved R6 35.7 mm to (148.7, 126.5), turned to 90 degrees
- moved R4 34.8 mm to (158.5, 123.8)
- moved R3 34.8 mm to (154.7, 123.8)
- moved R9 34.2 mm to (138.4, 126.5), turned to -90 degrees
- moved R12 33.9 mm to (144.5, 126.5), turned to 90 degrees
- moved J1 32.8 mm to (159.6, 113.8), turned to 0 degrees
- moved R10 32.1 mm to (140.5, 126.5), turned to 90 degrees
- moved J5 31.7 mm to (173.1, 118.2)
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Connections:
- C2 pad 1: Net-(D3-K) -> Net-(D1-A2)
- C4 pad 2: 5V -> 3v3
- D1 pad 2: Net-(D1-A) -> Net-(D1-A2)
- D3 pad 1: Net-(D3-K) -> Net-(D1-A2)
- F1 pad 2: Net-(D3-K) -> Net-(D1-A2)
- R10 pad 2: Net-(D10-A) -> GND
- R12 pad 2: Net-(D11-A) -> GND
- R35 pad 1: FLYWHEEL -> Coolant
- R35 pad 2: Net-(R35-Pad2) -> Engine Batt+
- R36 pad 2: FLYWHEEL -> OilPressure
- R37 pad 1: Net-(R35-Pad2) -> FLYWHEEL
- R37 pad 2: 5V -> 3v3
- R38 pad 2: Net-(R35-Pad2) -> FLYWHEEL
- R6 pad 2: Net-(D1-A) -> GND
- U1 pad 14: 1-Wire -> unconnected-(U1-GP10-Pad14)
- U1 pad 4: unconnected-(U1-GP0-Pad4) -> 1-Wire
- U2 pad 3: Net-(D3-K) -> Net-(D1-A2)
- U7 pad 1: Net-(R35-Pad2) -> FLYWHEEL
- U7 pad 8: 5V -> 3v3
Routing:
- net GND: track 619.2 -> 408.6 mm, vias 9 -> 4
- net 3v3: track 58.9 -> 129.8 mm, vias 2 -> 4
- net 5V: track 435.0 -> 366.4 mm, vias 5 -> 3
- net STOP: track 49.7 -> 8.83 mm
- net START: track 23.8 -> 50.4 mm
- net FLYWHEEL: track 102.8 -> 77.6 mm, vias 2 -> 0
- net GLOW: track 24.3 -> 45.2 mm
- net Net-(D1-A2): track 0.00 -> 20.6 mm
- net 1-Wire: track 77.1 -> 57.4 mm, vias 2 -> 1
- net Net-(U3-RXD): track 20.6 -> 2.45 mm
- net Net-(R35-Pad2): track 16.1 -> 0.00 mm
- net SDA: track 99.3 -> 83.8 mm, vias 0 -> 3
- net SCL3: track 24.5 -> 39.3 mm
- net Net-(D3-K): track 14.4 -> 0.00 mm
- net NTC3: track 34.8 -> 47.7 mm
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Other:
- board size 122.2 x 54.6 mm -> 108 x 47 mm
- board text added: "${REFERENCE}"

Commit message: Fixed some hardware problems
Parts:
- added D10: 1N47xxA 5v1, Diode_THT:D_T-1_P5.08mm_Horizontal, F.Cu at (85.7, 140.2)
- added D11: 1N47xxA 3v3, Diode_THT:D_T-1_P5.08mm_Horizontal, F.Cu at (138.6, 134.2)
- added D4: 1N47xxA 3v3, Diode_THT:D_T-1_P5.08mm_Horizontal, F.Cu at (138.7, 130.9)
- added D5: 1N47xxA 3v3, Diode_THT:D_T-1_P5.08mm_Horizontal, F.Cu at (138.6, 137.5)
- R10, R12, R6: value 2.2K -> 3K3
Connections:
- D2 pad 1: 5V -> 3v3
- J1 pad 2: 5V -> 3v3
- R2 pad 2: 5V -> 3v3
Routing:
- net 5V: track 366.4 -> 322.7 mm
- net 3v3: track 129.8 -> 173.3 mm
- net STOP: track 8.83 -> 23.4 mm
- net GND: track 408.6 -> 413.9 mm
- net START: track 50.4 -> 53.3 mm
- net Coolant: track 14.9 -> 17.4 mm, vias 1 -> 0
- net 1-Wire: track 57.4 -> 59.2 mm
- net GLOW: track 45.2 -> 46.3 mm

Commit message: Fixed some hardware problems
Parts:
- removed D4: 1N47xxA 3v3, Diode_THT:D_T-1_P5.08mm_Horizontal
- added D6: BAT46, Diode_SMD:Nexperia_CFP3_SOD-123W, F.Cu at (88.6, 139.7)
- C8: value 470nF -> 1nF
- D1: footprint Diode_SMD:D_SMA -> Diode_SMD:D_SMA-SMB_Universal_Handsoldering
- D10: value 1N47xxA 5v1 -> BAT46; footprint Diode_THT:D_T-1_P5.08mm_Horizontal -> Diode_SMD:Nexperia_CFP3_SOD-123W
- D11, D5: value 1N47xxA 3v3 -> BAT46; footprint Diode_THT:D_T-1_P5.08mm_Horizontal -> Diode_SMD:Nexperia_CFP3_SOD-123W
- D2, D3: footprint Diode_SMD:D_0805_2012Metric_Pad1.15x1.40mm_HandSolder -> Diode_SMD:D_SMA
- D7, D8: footprint Diode_SMD:D_SOD-123 -> Diode_SMD:D_SMA
- R13, R14, R7, R8: value 10K -> 4K7
- R35: footprint Resistor_SMD:R_0805_2012Metric_Pad1.20x1.40mm_HandSolder -> Resistor_THT:R_Axial_DIN0204_L3.6mm_D1.6mm_P5.08mm_Horizontal
- R38: value 220K -> 470K
- moved D10 60.5 mm to (143.4, 121.8), turned to -90 degrees
- moved D5 19.0 mm to (149.1, 121.8), turned to -90 degrees
- moved D11 14.7 mm to (146.3, 121.8), turned to -90 degrees
- moved J2 9.80 mm to (134.0, 129.8)
- moved R35 4.10 mm to (83.7, 139.6)
- moved R5 3.46 mm to (150.1, 126.4), turned to 90 degrees
- moved R9 2.74 mm to (141.1, 126.4), turned to 90 degrees
- moved R39 2.16 mm to (134.1, 123.7), turned to -90 degrees
- moved R11 2.01 mm to (144.4, 126.4), turned to 90 degrees
- moved R44 1.94 mm to (86.6, 128.5), turned to 90 degrees
- moved R12 1.78 mm to (146.3, 126.4), turned to -90 degrees
- moved R43 1.52 mm to (82.8, 123.5)
- moved R38 1.45 mm to (96.5, 121.8)
- moved R10 1.40 mm to (139.1, 126.4), turned to -90 degrees
- moved C8 1.30 mm to (86.0, 124.3)
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Connections:
- D10 pad 1: Coolant -> 3v3
- D10 pad 2: GND -> START
- D11 pad 1: GLOW -> 3v3
- D11 pad 2: GND -> GLOW
- D5 pad 1: STOP -> 3v3
- D5 pad 2: GND -> STOP
Routing:
- net GND: track 413.9 -> 465.1 mm, vias 4 -> 7
- net 3v3: track 173.3 -> 212.5 mm
- net 5V: track 322.7 -> 343.6 mm, vias 3 -> 4
- net STOP: track 23.4 -> 8.86 mm
- net Fuel: track 16.3 -> 22.0 mm
- net STOPCOIL: track 14.6 -> 19.6 mm
- net Net-(D7-K): track 25.2 -> 29.8 mm
- net Coolant: track 17.4 -> 13.3 mm
- net GLOWCOIL: track 15.1 -> 19.0 mm
- net GLOW: track 46.3 -> 49.4 mm
- net STARTCOIL: track 16.6 -> 19.4 mm
- net Net-(D1-A2): track 20.6 -> 18.0 mm
- net Engine Batt+: track 36.9 -> 35.0 mm, vias 2 -> 1
- net START: track 53.3 -> 55.0 mm
- net FLYWHEEL: track 77.6 -> 78.4 mm
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
Commit message: Fixed final hardware adjustments
Parts:
- D10, D11, D5, D6: footprint Diode_SMD:Nexperia_CFP3_SOD-123W -> Diode_SMD:D_SOD-123
- D7, D8: value SJ1 -> S1J
- R10, R12, R6: value 3K3 -> 4K7
- moved R2 13.2 mm to (175.6, 125.0), turned to 0 degrees
- moved D2 9.40 mm to (175.0, 122.3), turned to 180 degrees
- moved J5 3.72 mm to (170.7, 115.4), turned to 0 degrees
- turned R45 to -90 degrees
Connections:
- net Engine Batt+ renamed Engine Batt Switched +
Routing:
- net 1-Wire: track 59.2 -> 29.3 mm
- net 3v3: track 212.5 -> 191.0 mm
- net CAN-L: track 6.89 -> 11.8 mm
- net STOP: track 8.86 -> 11.0 mm
- net Engine Batt Switched +: track 35.0 -> 33.5 mm
- net CAN-H: track 7.42 -> 8.15 mm
- net GND: track 465.1 -> 465.6 mm
