File: pcb/esp32board/esp32board.kicad_sch (KiCad schematic)
At the start: 85 parts, among them J1 1Wire, J10 NTC5, J11 FuelLevel, J12 12V In, J13 Oil Pressure, J14 Engine, J15 Flywheel, J16 Relays, J5 CAN, J6 NTC1, J7 NTC2, J8 NTC3, J9 NTC4, Q1 BS170F, Q2 BS170F, U1 ESP32-C3-Waveshare, U2 AMS1117-5.0, U3 TJA1050, U4 ADS1115IDGS, U5 ADS1115IDGS, U6 ADS1115IDGS, U7 LM393

Commit message: Fixed some hardware problems, new board
Parts:
- removed D1, D10, D11: LED, LED_SMD:LED_0805_2012Metric_Pad1.15x1.40mm_HandSolder, symbol Device:LED
- added D1: SMAJ16CA, Diode_SMD:D_SMA, symbol Diode:SMAJ16CA
- added J2: V2_spare, Connector_PinHeader_2.54mm:PinHeader_1x01_P2.54mm_Vertical, symbol Connector:Conn_01x01_Pin
- Q1, Q2: value BS170F -> BSS138
- R35: value 2K2 -> 1K
- R36: value 3K3 -> 22K
- R42: value 4K7 -> 3K3
Connections:
- net 1-Wire: now also U1.4 (GP0); no longer U1.14 (GP10)
- net 3v3: now also C4.2, R37.2, U7.8 (V+)
- net 5V: no longer C4.2, R37.2, U7.8 (V+)
- net Coolant: now also R35.1
- net Engine Batt+: now also R35.2
- net FLYWHEEL: now also R37.1, R38.2, U7.1; no longer R35.1, R36.2
- net GND: now also R10.2, R12.2, R6.2, D1.1 (A1)
- net OilPressure: now also R36.2
- net V2: now also J2.1 (Pin_1)
- net at C2.1, D3.1 (K), F1.2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: now also D1.2 (A2)
- no-connect marks 10 -> 9
Other:
- note added: "10K Ok for 100KHz I2C Use 4K7 for 400KHz"
- note added: "The coolant sensor is fed from Engine Batt via a 1K resistor. Engine Batt+ terminal must be connected to the 1K resistor The onboard 1K pullup R35 should only be added if not external."
- note removed: "The coolant sensor is fed from Engine Batt via a 1K resistor. Engine Batt+ terminal must be connected to the 1K resistor"

Commit message: Fixed some hardware problems
Parts:
- added D10: 1N47xxA 5v1, Diode_THT:D_T-1_P5.08mm_Horizontal, symbol Diode:1N47xxA
- added D11, D4, D5: 1N47xxA 3v3, Diode_THT:D_T-1_P5.08mm_Horizontal, symbol Diode:1N47xxA
- R10, R12, R6: value 2.2K -> 3K3
Connections:
- net 3v3: now also D2.1 (K), J1.2 (Pin_2), R2.2
- net 5V: no longer D2.1 (K), J1.2 (Pin_2), R2.2
- net Coolant: now also D10.1 (K)
- net GLOW: now also D11.1 (K)
- net GND: now also D10.2 (A), D11.2 (A), D4.2 (A), D5.2 (A)
- net START: now also D4.1 (K)
- net STOP: now also D5.1 (K)

Commit message: Fixed some hardware problems
Parts:
- removed D10: 1N47xxA 5v1, Diode_THT:D_T-1_P5.08mm_Horizontal, symbol Diode:1N47xxA
- removed D11, D4, D5: 1N47xxA 3v3, Diode_THT:D_T-1_P5.08mm_Horizontal, symbol Diode:1N47xxA
- added D10, D11, D5, D6: BAT46, Diode_SMD:Nexperia_CFP3_SOD-123W, symbol Diode:BAT46
- C8: value 470nF -> 1nF
- D1: footprint Diode_SMD:D_SMA -> Diode_SMD:D_SMA-SMB_Universal_Handsoldering
- D2, D3: footprint Diode_SMD:D_0805_2012Metric_Pad1.15x1.40mm_HandSolder -> Diode_SMD:D_SMA
- D7, D8: footprint Diode_SMD:D_SOD-123 -> Diode_SMD:D_SMA
- R13, R14, R7, R8: value 10K -> 4K7
- R35: footprint Resistor_SMD:R_0805_2012Metric_Pad1.20x1.40mm_HandSolder -> Resistor_THT:R_Axial_DIN0204_L3.6mm_D1.6mm_P5.08mm_Horizontal
- R38: value 220K -> 470K
Connections:
- net 3v3: now also D10.1 (K), D11.1 (K), D5.1 (K)
- net 5V: now also D6.1 (K)
- net Coolant: now also D6.2 (A)
- net GLOW: now also D11.2 (A)
- net START: now also D10.2 (A)
- net STOP: now also D5.2 (A)
- no-connect marks 9 -> 10

Commit message: Fixed final hardware adjustments
Parts:
- D10, D11, D5, D6: footprint Diode_SMD:Nexperia_CFP3_SOD-123W -> Diode_SMD:D_SOD-123
- D7, D8: value SJ1 -> S1J
- R10, R12, R6: value 3K3 -> 4K7
Connections:
- net Engine Batt+ renamed Engine Batt Switched +
Changed lines of the file:
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@@
 		)
 	)
-	(global_label "Engine Batt+"
+	(global_label "Engine Batt Switched +"
 		(shape input)
-		(at 256.54 137.16 0)
+		(at 240.03 116.84 180)
 		(fields_autoplaced yes)
 		(effects
@@
 				(size 1.27 1.27)
 			)
-			(justify left)
+			(justify right)
 		)
 		(property "Intersheetrefs" "${INTERSHEET_REFS}"
-			(at 272.225 137.16 0)
+			(at 214.0641 116.84 0)
 			(effects
 				(font
 					(size 1.27 1.27)
 				)
-				(justify left)
+				(justify right)
 				(hide yes)
 			)
@@
 		)
 	)
+	(global_label "Engine Batt Switched +"
+		(shape input)
+		(at 256.54 137.16 0)
+		(fields_autoplaced yes)
+		(effects
+			(font
+				(size 1.27 1.27)
+			)
+			(justify left)
+		)
+		(property "Intersheetrefs" "${INTERSHEET_REFS}"
+			(at 282.5059 137.16 0)
+			(effects
+				(font
+					(size 1.27 1.27)
+				)
+				(justify left)
+				(hide yes)
+			)
+		)
+	)
 	(global_label "5V"
 		(shape input)
@@
 		)
 	)
-	(global_label "Engine Batt+"
+	(global_label "Engine Batt Switched +"
 		(shape output)
 		(at 234.95 105.41 180)
@@
 		)
 		(property "Intersheetrefs" "${INTERSHEET_REFS}"
-			(at 219.265 105.41 0)
+			(at 208.9841 105.41 0)
 			(effects
 				(font
@@
 		)
 	)
-	(global_label "Engine Batt+"
-		(shape input)
-		(at 240.03 116.84 180)
-		(fields_autoplaced yes)
-		(effects
-			(font
-				(size 1.27 1.27)
-			)
-			(justify right)
-		)
-		(property "Intersheetrefs" "${INTERSHEET_REFS}"
-			(at 224.345 116.84 0)
-			(effects
-				(font
-					(size 1.27 1.27)
-				)
-				(justify right)
-				(hide yes)
-			)
-		)
-	)
 	(global_label "CAN-L"
 		(shape bidirectional)
@@
 			)
 		)
-		(property "Value" "SJ1"
+		(property "Value" "S1J"
 			(at 217.17 38.735 90)
 			(effects
@@
 			)
 		)
-		(property "Value" "SJ1"
+		(property "Value" "S1J"
 			(at 208.28 40.005 90)
 			(effects
@@
 	)
 	(symbol
-		(lib_name "GND_1")
-		(lib_id "power:GND")
-		(at 250.19 124.46 0)
-		(unit 1)
-		(exclude_from_sim no)
-		(in_bom yes)
-		(on_board yes)
-		(dnp no)
-		(fields_autoplaced yes)
-		(property "Reference" "#PWR039"
-			(at 250.19 130.81 0)
-			(effects
-				(font
-					(size 1.27 1.27)
-				)
-				(hide yes)
-			)
-		)
-		(property "Value" "GND"
-			(at 250.19 129.54 0)
-			(effects
-				(font
-					(size 1.27 1.27)
-				)
-			)
-		)
-		(property "Footprint" ""
-			(at 250.19 124.46 0)
-			(effects
-				(font
-					(size 1.27 1.27)
-				)
-				(hide yes)
-			)
-		)
-		(property "Datasheet" ""
-			(at 250.19 124.46 0)
-			(effects
-				(font
-					(size 1.27 1.27)
-				)
-				(hide yes)
-			)
-		)
-		(property "Description" "Power symbol creates a global label with name \"GND\" , ground"
-			(at 250.19 124.46 0)
-			(effects
-				(font
-					(size 1.27 1.27)
-				)
-				(hide yes)
-			)
-		)
-		(pin "1"
-		)
-		(instances
-			(project "esp32board"
-				(path "/461a08a1-c6de-4673-bbd4-d74d528c254e"
-					(reference "#PWR039")
-					(unit 1)
-				)
-			)
-		)
-	)
-	(symbol
 		(lib_id "Connector_Generic:Conn_01x04")
 		(at 240.03 100.33 0)
@@
 			)
 		)
-		(property "Footprint" "Diode_SMD:Nexperia_CFP3_SOD-123W"
+		(property "Footprint" "Diode_SMD:D_SOD-123"
 			(at 245.745 113.03 0)
 			(effects
@@
 			)
 		)
-		(property "Footprint" "Diode_SMD:Nexperia_CFP3_SOD-123W"
+		(property "Footprint" "Diode_SMD:D_SOD-123"
 			(at 78.105 146.05 0)
 			(effects
@@
 			)
 		)
-		(property "Value" "3K3"
+		(property "Value" "4K7"
 			(at 81.28 154.9399 0)
 			(effects
@@
 			)
 		)
-		(property "Footprint" "Diode_SMD:Nexperia_CFP3_SOD-123W"
+		(property "Footprint" "Diode_SMD:D_SOD-123"
 			(at 94.615 146.05 0)
 			(effects
@@
 			)
 		)
-		(property "Value" "3K3"
+		(property "Value" "4K7"
 			(at 66.04 154.9399 0)
 			(effects
@@
 			)
 		)
-		(property "Value" "3K3"
+		(property "Value" "4K7"
 			(at 95.25 154.9399 0)
 			(effects
@@
 			)
 		)
-		(property "Footprint" "Diode_SMD:Nexperia_CFP3_SOD-123W"
+		(property "Footprint" "Diode_SMD:D_SOD-123"
 			(at 64.135 146.05 0)
 			(effects
